Commit message: Obstacle in URDF

File: roy_dmp/urdf/test_d435i_camera.urdf.xacro (robot description, xacro)
@@ -22,5 +22,5 @@
       <parent link="base_link"/>
       <child link="camera_base_link"/>
-      <origin xyz="0.5 0 0" rpy="0 0 0"/>
+      <origin xyz="0.5 0.5 0.5" rpy="0 0.75 -2.0"/>
     </joint>
   </xacro:unless>

File: roy_dmp/urdf/ur3.xacro (robot description, xacro)
@@ -10,4 +10,5 @@
   <xacro:arg name="safety_pos_margin" default="0.15"/>
   <xacro:arg name="safety_k_position" default="20"/>
+  <xacro:arg name="obstacle_urdf" default="none"/>
   <xacro:arg name="use_cam" default="true"/>
   <xacro:arg name="use_cam_tool" default="false"/>
@@ -26,3 +27,8 @@
     <xacro:include filename="$(arg camera_urdf)"/>
   </xacro:if>
+<!-- obstacle -->
+<xacro:property name="obstacle_urdf" value="$(arg obstacle_urdf)"/>
+  <xacro:unless value="${obstacle_urdf == 'none'}">
+    <xacro:include filename="$(arg obstacle_urdf)"/>
+  </xacro:unless>
 </robot>
