Commit message: remove gazebo ground

File: roy_dmp/urdf/cube.xacro (robot description, xacro)
@@ -11,4 +11,7 @@
           <box size="${size} ${size} ${size}"/>
       </geometry>
+      <material name="cube_blue">
+          <color rgba="0 0 1 1"/>
+      </material>
     </visual>
     <collision>
@@ -19,7 +22,4 @@
     </collision>
     </link>
-    <gazebo reference="cube0">
-      <material>Gazebo/Blue</material>
-    </gazebo>
     <joint name="cube0_joint" type="fixed">
       <parent link="base_link" />
