Commit message: real cam & robot setup

File: roy_dmp/urdf/ur3.xacro (robot description, xacro)
@@ -12,4 +12,5 @@
   <xacro:arg name="obstacle_urdf" default="none"/>
   <xacro:arg name="use_cam" default="true"/>
+  <xacro:arg name="sim_cam" default="true"/>
   <xacro:arg name="use_cam_tool" default="false"/>
   <xacro:arg name="camera_urdf" default=""/>
@@ -20,4 +21,5 @@
   <!-- camera -->
   <xacro:property name="use_cam" value="$(arg use_cam)"/>
+  <xacro:property name="sim_cam" value="$(arg sim_cam)"/>
   <xacro:if value="${use_cam}">
     <xacro:arg name="name" default="camera" />
@@ -27,5 +29,10 @@
     <xacro:arg name="add_plug" default="false" />
     <xacro:arg name="parent" default="camera_base_link" />
-    <xacro:include filename="$(arg camera_urdf)"/>
+    <xacro:if value="${sim_cam}">
+    	<xacro:include filename="$(arg camera_urdf)"/>
+    </xacro:if>
+    <xacro:unless value="${sim_cam}">
+    	<xacro:include filename="$(find roy_dmp)/urdf/d435_camera.urdf.xacro"/>
+    </xacro:unless>
   </xacro:if>
 <!-- obstacle -->

Commit message: tool model update

File: roy_dmp/urdf/ur3.xacro (robot description, xacro)
@@ -15,8 +15,12 @@
   <xacro:arg name="use_cam_tool" default="false"/>
   <xacro:arg name="camera_urdf" default=""/>
+  <xacro:property name="M_PI" value="3.14159265359" />
+  <xacro:property name="robot_prefix" value=""/>
   <!-- ur3 -->
   <xacro:include filename="$(find ur_gazebo)/urdf/ur.xacro"/>
-  <!-- tool -->
-  <xacro:include filename="$(find roy_dmp)/urdf/tool.xacro"/>
+  <!-- rg2 gripper -->
+  <!--<xacro:include filename="$(find roy_dmp)/urdf/tool.xacro"/>-->
+  <xacro:include filename="$(find roy_dmp)/urdf/rg2.urdf.xacro" />
+  <xacro:rg2 prefix="${robot_prefix}"/>
   <!-- base -->
   <xacro:include filename="$(find roy_dmp)/urdf/base.xacro"/>
