Commit message: camera position update

File: roy_dmp/urdf/test_d435_camera.urdf.xacro (robot description, xacro)
@@ -22,5 +22,5 @@
       <parent link="base_link"/>
       <child link="camera_base_link"/>
-      <origin xyz="0.5 0.5 0.5" rpy="0 0.75 -2.0"/>
+      <origin xyz="-0.4 0.4 0.25" rpy="0 0.0 -0.5"/>
     </joint>
   </xacro:unless>
