Commit message: updated tool 2

File: roy_dmp/urdf/rg2.urdf.xacro (robot description, xacro)
@@ -6,5 +6,5 @@
     <!-- rg2 joint -->
     <joint name="rg2_joint" type="fixed">
-      <origin xyz="0.01 0 0" rpy="0 0 0" />
+      <origin xyz="0.01 0 0" rpy="-${M_PI/2} 0 0" />
       <parent link="${prefix}flange"/>
       <child link="${prefix}rg2_body_link"/>
