Commit message: camera launch unification

File: roy_dmp/urdf/d435_camera.urdf.xacro (robot description, xacro)
@@ -8,5 +8,5 @@
   <xacro:arg name="sim_cam" default="false" />
   <xacro:arg name="use_mesh" default="true" />
-  <xacro:arg name="publish_pointcloud" default="false" />
+  <xacro:arg name="publish_pointcloud" default="false"/>
   <xacro:property name="sim_cam" value="$(arg sim_cam)" />
   <xacro:if value="${sim_cam}">
@@ -16,5 +16,5 @@
     <xacro:arg name="use_nominal_extrinsics" default="false"/>
   </xacro:unless>
-  <xacro:include filename="$(find realsense2_description)/urdf/_d435.urdf.xacro" />
+  <xacro:include filename="$(find roy_dmp)/urdf/_d435.urdf.xacro" />
   <link name="$(arg parent)" />
   <xacro:property name="use_cam_tool" value="$(arg use_cam_tool)" />
@@ -38,5 +38,5 @@
       <parent link="cam_support_base_link"/>
       <child link="cam_support_1_link"/>
-      <origin xyz="0 0 0.4" rpy="0 0 0"/>
+      <origin xyz="0.01931 0 0.61" rpy="0 0 0"/>
     </joint>
     <joint name="cam_joint_3" type="fixed">
@@ -48,8 +48,8 @@
       <parent link="cam_support_2_link"/>
       <child link="camera_base_link"/>
-      <origin xyz="0 0.019 -0.012" rpy="0 0 0"/>
+      <origin xyz="0.019 0.0 -0.012" rpy="0 0 0"/>
     </joint>
   </xacro:unless>
-  <xacro:sensor_d435 parent="$(arg parent)" use_nominal_extrinsics="$(arg use_nominal_extrinsics)" add_plug="$(arg add_plug)" use_mesh="$(arg use_mesh)" name="$(arg name)" topics_ns="$(arg topics_ns)" publish_pointcloud="$(arg publish_pointcloud)">
+  <xacro:sensor_d435 parent="$(arg parent)" gazebo="$(arg sim_cam)" use_nominal_extrinsics="$(arg use_nominal_extrinsics)" add_plug="$(arg add_plug)" use_mesh="$(arg use_mesh)" name="$(arg name)" topics_ns="$(arg topics_ns)" publish_pointcloud="$(arg publish_pointcloud)">
     <origin xyz="0 0 0" rpy="0 0 0"/>
   </xacro:sensor_d435>

File: roy_dmp/urdf/ur3.xacro (robot description, xacro)
@@ -10,10 +10,13 @@
   <xacro:arg name="safety_pos_margin" default="0.15"/>
   <xacro:arg name="safety_k_position" default="20"/>
-  <xacro:arg name="obstacle_urdf" default="none"/>
   <xacro:arg name="use_cam" default="true"/>
   <xacro:arg name="sim_cam" default="true"/>
   <xacro:arg name="use_cam_tool" default="false"/>
   <xacro:arg name="camera_urdf" default=""/>
-  <xacro:arg name="sim" default="false" />
+  <xacro:arg name="name" default="camera" />
+  <xacro:arg name="topics_ns" default="camera" />
+  <xacro:arg name="publish_pointcloud" default="true" />
+  <xacro:arg name="add_plug" default="false" />
+  <xacro:arg name="parent" default="camera_base_link" />
   <xacro:property name="M_PI" value="3.14159265359" />
   <xacro:property name="robot_prefix" value=""/>
@@ -28,23 +31,6 @@
   <!-- camera -->
   <xacro:property name="use_cam" value="$(arg use_cam)"/>
-  <xacro:property name="sim_cam" value="$(arg sim_cam)"/>
   <xacro:if value="${use_cam}">
-    <xacro:arg name="name" default="camera" />
-    <xacro:arg name="topics_ns" default="camera" />
-    <xacro:arg name="use_nominal_extrinsics" default="true" />
-    <xacro:arg name="publish_pointcloud" default="true" />
-    <xacro:arg name="add_plug" default="false" />
-    <xacro:arg name="parent" default="camera_base_link" />
-    <xacro:if value="${sim_cam}">
     <xacro:include filename="$(arg camera_urdf)"/>
-    </xacro:if>
-    <xacro:unless value="${sim_cam}">
-    	<xacro:include filename="$(find roy_dmp)/urdf/d435_camera.urdf.xacro"/>
-    </xacro:unless>
   </xacro:if>
-<!-- obstacle -->
-<xacro:property name="obstacle_urdf" value="$(arg obstacle_urdf)"/>
-  <xacro:unless value="${obstacle_urdf == 'none'}">
-    <xacro:include filename="$(arg obstacle_urdf)"/>
-  </xacro:unless>
 </robot>

Commit message: camera off adjust + safety check val + cpp tidy

File: roy_dmp/urdf/d435_camera.urdf.xacro (robot description, xacro)
@@ -33,5 +33,5 @@
       <parent link="base_link"/>
       <child link="cam_support_base_link"/>
-      <origin xyz="-0.55 0.8 0" rpy="0 0 -0.7854"/>
+      <origin xyz="-0.55 0.77 0" rpy="0 0 -0.7854"/>
     </joint>
     <joint name="cam_joint_2" type="fixed">
