Commit message: add virtual walls

File: roy_dmp/urdf/base.xacro (robot description, xacro)
@@ -1,7 +1,7 @@
 <?xml version="1.0"?>
 <robot name="base_plate" xmlns:xacro="http://ros.org/wiki/xacro">
-<link name="base_plate">
+  <link name="base_plate">
     <visual>
-    <origin xyz="0 0 -0.01"/>
+      <origin xyz="0 0 -0.01"/>
       <geometry>
           <box size="1.0 1.0 0.02"/>
@@ -12,45 +12,67 @@
     </visual>
     <collision>
-    <origin xyz="0 0 -0.01"/>
+      <origin xyz="0 0 -0.01"/>
       <geometry>
         <box size="1.0 1.0 0.02"/>
       </geometry>
     </collision>
-    </link>
-    <joint name="base_joint" type="fixed">
-      <parent link="base_link" />
-      <child link = "base_plate" />
-      <origin xyz="0 0 0" rpy="0 0 0" />
-    </joint>
-    </robot>
-<!-- <xacro:macro name="cube" params="">
-<xacro:property name="size" value="0.1"/>
-  <link name="cube_link">
-    <inertial>
-      <origin xyz="${size/2.0} ${size/2.0} ${size/2.0}" />
-      <mass value="1.0" />
-      <inertia  ixx="1.0" ixy="0.0"  ixz="1.0"  iyy="1.0"  iyz="1.0"  izz="1.0" />
-    </inertial>
-    <visual>
-      <origin xyz="${size/2.0} ${size/2.0} ${size/2.0}"/>
+  </link>
+  <joint name="base_joint" type="fixed">
+    <parent link="base_link" />
+    <child link = "base_plate" />
+    <origin xyz="0.3 0 0" rpy="0 0 0" />
+  </joint>
+  <!-- Virtual safety walls -->
+  <link name="wall1_link">
+    <collision>
+      <origin xyz="0 0 0"/>
       <geometry>
-        <box size="${size} ${size} ${size}" />
-      </geometry>
-    </visual>
-    <collision>
-      <origin xyz="${size/2.0} ${size/2.0} ${size/2.0}"/>
-      <geometry>
-        <box size="${size} ${size} ${size}" />
+        <box size="1.0 1.0 0.02"/>
       </geometry>
     </collision>
   </link>
-  <gazebo reference="cube">
-  <material>Gazebo/Blue</material>
-  </gazebo>
-  </xacro:macro>
-    <joint name="cube_joint" type="fixed">
-      <parent link="base_link"/>
-      <child link="cube_link"/>
-      <origin xyz="0.2 0.2 0.2" rpy="0 0.0 0.0"/>
+  <joint name="wall1_joint" type="fixed">
+    <parent link="base_plate" />
+    <child link = "wall1_link" />
+    <origin xyz="0 -0.5 0.48" rpy="1.57079632679 0 0" />
   </joint>
--->
+  <link name="wall2_link">
+    <collision>
+      <origin xyz="0 0 0"/>
+      <geometry>
+        <box size="1.0 1.0 0.02"/>
+      </geometry>
+    </collision>
+  </link>
+  <joint name="wall2_joint" type="fixed">
+    <parent link="base_plate" />
+    <child link = "wall2_link" />
+    <origin xyz="0.5 0 0.48" rpy="1.57079632679 0 1.57079632679" />
+  </joint>
+  <link name="wall3_link">
+    <collision>
+      <origin xyz="0 0 0"/>
+      <geometry>
+        <box size="1.0 1.0 0.02"/>
+      </geometry>
+    </collision>
+  </link>
+  <joint name="wall3_joint" type="fixed">
+    <parent link="base_plate" />
+    <child link = "wall3_link" />
+    <origin xyz="0 0.5 0.48" rpy="1.57079632679 0 0" />
+  </joint>
+  <link name="wall4_link">
+    <collision>
+      <origin xyz="0 0 0"/>
+      <geometry>
+        <box size="1.0 1.0 0.02"/>
+      </geometry>
+    </collision>
+  </link>
+  <joint name="wall4_joint" type="fixed">
+    <parent link="base_plate" />
+    <child link = "wall4_link" />
+    <origin xyz="-0.5 0 0.48" rpy="1.57079632679 0 1.57079632679" />
+  </joint>
+</robot>

Commit message: robot + cam definition update

File: roy_dmp/urdf/base.xacro (robot description, xacro)
@@ -21,5 +21,5 @@
     <parent link="base_link" />
     <child link = "base_plate" />
-    <origin xyz="0.3 0 0" rpy="0 0 0" />
+    <origin xyz="0 0.25 0" rpy="0 0 0" />
   </joint>
   <!-- Virtual safety walls -->

File: roy_dmp/urdf/d435_camera.urdf.xacro (robot description, xacro)
@@ -23,5 +23,5 @@
       <parent link="base_link"/>
       <child link="camera_base_link"/>
-      <origin xyz="0.5 0.5 0.5" rpy="0 0.75 -2.0"/>
+      <origin xyz="-0.4 0.4 0.25" rpy="0 0.0 -0.5"/>
     </joint>
   </xacro:unless>

File: roy_dmp/urdf/tool.xacro (robot description, xacro)
@@ -21,5 +21,5 @@
     <parent link="wrist_3_link"/>
     <child link="tool_claw"/>
-    <origin xyz="0 0 0.11" rpy="0 -1.5707 0"/>
+    <origin xyz="0 0 0.11" rpy="-1.5707 -1.5707 0"/>
   </joint>
 </robot>

File: roy_dmp/urdf/ur3.xacro (robot description, xacro)
@@ -32,5 +32,5 @@
     <xacro:arg name="parent" default="camera_base_link" />
     <xacro:if value="${sim_cam}">
-    	<xacro:include filename="$(arg camera_urdf)"/>
+    <xacro:include filename="$(arg camera_urdf)"/>
     </xacro:if>
     <xacro:unless value="${sim_cam}">

Commit message: base + cam urdf setup update

File: roy_dmp/urdf/base.xacro (robot description, xacro)
@@ -21,5 +21,5 @@
     <parent link="base_link" />
     <child link = "base_plate" />
-    <origin xyz="0 0.25 0" rpy="0 0 0" />
+    <origin xyz="-0.05 0.3 0" rpy="0 0 0" />
   </joint>
   <!-- Virtual safety walls -->

File: roy_dmp/urdf/d435_camera.urdf.xacro (robot description, xacro)
@@ -23,5 +23,5 @@
       <parent link="base_link"/>
       <child link="camera_base_link"/>
-      <origin xyz="-0.4 0.4 0.25" rpy="0 0.0 -0.5"/>
+      <origin xyz="-0.5 0.7 0.18" rpy="0 0.0 -1.0"/>
     </joint>
   </xacro:unless>

Commit message: robot + cam + base redefintion

File: roy_dmp/urdf/base.xacro (robot description, xacro)
@@ -1,4 +1,5 @@
 <?xml version="1.0"?>
 <robot name="base_plate" xmlns:xacro="http://ros.org/wiki/xacro">
+  <xacro:arg name="sim" default="true" />
   <link name="base_plate">
     <visual>
@@ -24,55 +25,58 @@
   </joint>
   <!-- Virtual safety walls -->
-  <link name="wall1_link">
-    <collision>
-      <origin xyz="0 0 0"/>
-      <geometry>
-        <box size="1.0 1.0 0.02"/>
-      </geometry>
-    </collision>
-  </link>
-  <joint name="wall1_joint" type="fixed">
-    <parent link="base_plate" />
-    <child link = "wall1_link" />
-    <origin xyz="0 -0.5 0.48" rpy="1.57079632679 0 0" />
-  </joint>
-  <link name="wall2_link">
-    <collision>
-      <origin xyz="0 0 0"/>
-      <geometry>
-        <box size="1.0 1.0 0.02"/>
-      </geometry>
-    </collision>
-  </link>
-  <joint name="wall2_joint" type="fixed">
-    <parent link="base_plate" />
-    <child link = "wall2_link" />
-    <origin xyz="0.5 0 0.48" rpy="1.57079632679 0 1.57079632679" />
-  </joint>
-  <link name="wall3_link">
-    <collision>
-      <origin xyz="0 0 0"/>
-      <geometry>
-        <box size="1.0 1.0 0.02"/>
-      </geometry>
-    </collision>
-  </link>
-  <joint name="wall3_joint" type="fixed">
-    <parent link="base_plate" />
-    <child link = "wall3_link" />
-    <origin xyz="0 0.5 0.48" rpy="1.57079632679 0 0" />
-  </joint>
-  <link name="wall4_link">
-    <collision>
-      <origin xyz="0 0 0"/>
-      <geometry>
-        <box size="1.0 1.0 0.02"/>
-      </geometry>
-    </collision>
-  </link>
-  <joint name="wall4_joint" type="fixed">
-    <parent link="base_plate" />
-    <child link = "wall4_link" />
-    <origin xyz="-0.5 0 0.48" rpy="1.57079632679 0 1.57079632679" />
-  </joint>
+  <xacro:property name="sim" value="$(arg sim)" />
+  <xacro:unless value="${sim}">
+    <link name="wall1_link">
+      <collision>
+        <origin xyz="0 0 0"/>
+        <geometry>
+          <box size="1.0 1.0 0.02"/>
+        </geometry>
+      </collision>
+    </link>
+    <joint name="wall1_joint" type="fixed">
+      <parent link="base_plate" />
+      <child link = "wall1_link" />
+      <origin xyz="0 -0.5 0.48" rpy="1.57079632679 0 0" />
+    </joint>
+    <link name="wall2_link">
+      <collision>
+        <origin xyz="0 0 0"/>
+        <geometry>
+          <box size="1.0 1.0 0.02"/>
+        </geometry>
+      </collision>
+    </link>
+    <joint name="wall2_joint" type="fixed">
+      <parent link="base_plate" />
+      <child link = "wall2_link" />
+      <origin xyz="0.5 0 0.48" rpy="1.57079632679 0 1.57079632679" />
+    </joint>
+    <link name="wall3_link">
+      <collision>
+        <origin xyz="0 0 0"/>
+        <geometry>
+          <box size="1.0 1.0 0.02"/>
+        </geometry>
+      </collision>
+    </link>
+    <joint name="wall3_joint" type="fixed">
+      <parent link="base_plate" />
+      <child link = "wall3_link" />
+      <origin xyz="0 0.5 0.48" rpy="1.57079632679 0 0" />
+    </joint>
+    <link name="wall4_link">
+      <collision>
+        <origin xyz="0 0 0"/>
+        <geometry>
+          <box size="1.0 1.0 0.02"/>
+        </geometry>
+      </collision>
+    </link>
+    <joint name="wall4_joint" type="fixed">
+      <parent link="base_plate" />
+      <child link = "wall4_link" />
+      <origin xyz="-0.5 0 0.48" rpy="1.57079632679 0 1.57079632679" />
+    </joint>
+  </xacro:unless>
 </robot>

File: roy_dmp/urdf/d435_camera.urdf.xacro (robot description, xacro)
@@ -1,12 +1,19 @@
 <?xml version="1.0"?>
 <robot name="realsense2_camera" xmlns:xacro="http://ros.org/wiki/xacro">
-  <xacro:arg name="use_nominal_extrinsics" default="false"/>
+  <xacro:arg name="use_cam_tool" default="false" />
+  <xacro:arg name="name" default="camera" />
   <xacro:arg name="add_plug" default="false" />
-  <xacro:arg name="use_mesh" default="true" />
-  <xacro:arg name="name" default="camera" />
   <xacro:arg name="parent" default="camera_base_link" />
   <xacro:arg name="topics_ns" default="camera" />
+  <xacro:arg name="sim_cam" default="false" />
+  <xacro:arg name="use_mesh" default="true" />
   <xacro:arg name="publish_pointcloud" default="false" />
-  <xacro:arg name="use_cam_tool" default="false" />
+  <xacro:property name="sim_cam" value="$(arg sim_cam)" />
+  <xacro:if value="${sim_cam}">
+    <xacro:arg name="use_nominal_extrinsics" default="true"/>
+  </xacro:if>
+  <xacro:unless value="${sim_cam}">
+    <xacro:arg name="use_nominal_extrinsics" default="false"/>
+  </xacro:unless>
   <xacro:include filename="$(find realsense2_description)/urdf/_d435.urdf.xacro" />
   <link name="$(arg parent)" />
@@ -20,8 +27,26 @@
   </xacro:if>
   <xacro:unless value="${use_cam_tool}">
-    <joint name="cam_tool" type="fixed">
+    <link name="cam_support_base_link" />
+    <link name="cam_support_1_link" />
+    <link name="cam_support_2_link" />
+    <joint name="cam_joint_1" type="fixed">
       <parent link="base_link"/>
+      <child link="cam_support_base_link"/>
+      <origin xyz="-0.55 0.8 0" rpy="0 0 -0.7854"/>
+    </joint>
+    <joint name="cam_joint_2" type="fixed">
+      <parent link="cam_support_base_link"/>
+      <child link="cam_support_1_link"/>
+      <origin xyz="0 0 0.4" rpy="0 0 0"/>
+    </joint>
+    <joint name="cam_joint_3" type="fixed">
+      <parent link="cam_support_1_link"/>
+      <child link="cam_support_2_link"/>
+      <origin xyz="0 0 0" rpy="0 0.7854 0"/>
+    </joint>
+    <joint name="cam_joint_4" type="fixed">
+      <parent link="cam_support_2_link"/>
       <child link="camera_base_link"/>
-      <origin xyz="-0.5 0.7 0.18" rpy="0 0.0 -1.0"/>
+      <origin xyz="0 0.019 -0.012" rpy="0 0 0"/>
     </joint>
   </xacro:unless>

File: roy_dmp/urdf/rg2.urdf.xacro (robot description, xacro)
@@ -2,4 +2,5 @@
 <!-- xacro for rg2 mounted on the manipulator -->
 <robot name="rg2" xmlns:xacro="http://ros.org/wiki/xacro">
+  <xacro:property name="M_PI" value="3.14159265359" />
   <xacro:macro name="rg2" params="prefix">
     <!--TODO remove screws from tool collision stl-->

File: roy_dmp/urdf/ur3.xacro (robot description, xacro)
@@ -15,4 +15,5 @@
   <xacro:arg name="use_cam_tool" default="false"/>
   <xacro:arg name="camera_urdf" default=""/>
+  <xacro:arg name="sim" default="false" />
   <xacro:property name="M_PI" value="3.14159265359" />
   <xacro:property name="robot_prefix" value=""/>

Commit message: collision real-time safe stop v1

File: roy_dmp/urdf/base.xacro (robot description, xacro)
@@ -22,5 +22,5 @@
     <parent link="base_link" />
     <child link = "base_plate" />
-    <origin xyz="-0.05 0.3 0" rpy="0 0 0" />
+    <origin xyz="-0.05 0.3 -0.001" rpy="0 0 0" />
   </joint>
   <!-- Virtual safety walls -->

Commit message: avoidance working in real robot

File: roy_dmp/urdf/base.xacro (robot description, xacro)
@@ -23,4 +23,26 @@
     <child link = "base_plate" />
     <origin xyz="-0.05 0.3 -0.001" rpy="0 0 0" />
+  </joint>
+  <link name="light_link">
+		<visual>
+			<origin xyz="0 0 0" rpy="0 0 0"/>
+			<geometry>
+				<cylinder length="0.3" radius="0.03"/>
+			</geometry>
+			<material name="light_white">
+          <color rgba="1 1 1 1"/>
+      </material>
+		</visual>
+		<collision>
+			<origin xyz="0 0 0" rpy="0 0 0"/>
+			<geometry>
+				<cylinder length="0.3" radius="0.03"/>
+			</geometry>
+		</collision>
+  </link>
+  <joint name="light_joint" type="fixed">
+    <parent link="base_plate" />
+    <child link = "light_link" />
+    <origin xyz="0.45 -0.45 0.16" rpy="0 0 0" />
   </joint>
   <!-- Virtual safety walls -->

File: roy_dmp/urdf/rg2.urdf.xacro (robot description, xacro)
@@ -7,5 +7,5 @@
     <!-- rg2 joint -->
     <joint name="rg2_joint" type="fixed">
-      <origin xyz="0.01 0 0" rpy="-${M_PI/2} 0 0" />
+      <origin xyz="0.005 0 0" rpy="-${M_PI/2} 0 0" />
       <parent link="${prefix}flange"/>
       <child link="${prefix}rg2_body_link"/>
